File: CustomSTM32H735Board/KiCADFiles/CustomSTM32H735Board/CustomSTM32H735Board.kicad_sch (KiCad schematic)
At the start: 57 parts, among them J1 Conn_01x03_Socket, J2 Conn_02x10_Odd_Even, J3 FTSH-105-01-L-DV-K, J4 FLE-125-01-G-DV, SW1 SW_Omron_B3FS, U1 STM32H735IGT6, X1 NSC5004A-25M

Commit message: more work on schematics
Parts:
- removed C13, C15: 4.7uF low ESR, Capacitor_SMD:C_0805_2012Metric_Pad1.18x1.45mm_HandSolder, symbol Device:C
- removed R10: 5k1, Resistor_SMD:R_0805_2012Metric_Pad1.20x1.40mm_HandSolder, symbol Device:R
- removed R11: R, Resistor_SMD:R_0805_2012Metric_Pad1.20x1.40mm_HandSolder, symbol Device:R
- removed U1: STM32H735IGT6, Private:LQFP176_STM32H735IGT6_STM-M, symbol Private:STM32H735IGT6
- added C? (x2): 4.7uF low ESR, Capacitor_SMD:C_0805_2012Metric_Pad1.18x1.45mm_HandSolder, symbol Device:C
- added R?: 1k, Resistor_SMD:R_0805_2012Metric_Pad1.20x1.40mm_HandSolder, symbol Device:R
- added R?: 5k1, Resistor_SMD:R_0805_2012Metric_Pad1.20x1.40mm_HandSolder, symbol Device:R
- added U? (x2): STM32H735IGT6, Private:LQFP176_STM32H735IGT6_STM-M, symbol Private:STM32H735IGT6
Connections:
- net +3.3V: now also R?.2, U?.105, U?.113, U?.126, U?.13, U?.136, U?.152, U?.160, U?.176, U?.25, U?.44, U?.48, U?.65, U?.7, U?.71, U?.8, U?.84, U?.92, U?.99
- net BOOT0: now also R?.1, U?.167
- net GND: now also C?.1, C?.1, R?.2, U?.100, U?.106, U?.112, U?.119, U?.12, U?.121, U?.134, U?.137, U?.151, U?.159, U?.173, U?.24, U?.38, U?.45, U?.47, U?.6, U?.64, U?.70, U?.81, U?.83, U?.93
- net NRST: now also U?.33
- net PA0: now also U?.41 (PA0-UART4_TX)
- net PA1: now also U?.42 (PA1-LTDC_R2)
- net PA10: now also U?.129 (PA10-LTDC_B1)
- net PA11: now also U?.130 (PA11-LTDC_R4)
- net PA13: now also U?.132 (PA13(JTMS/SWDIO)-DEBUG_JTMS-SWDIO)
- net PA14: now also U?.138 (PA14(JTCK/SWCLK)-DEBUG_JTCK-SWCLK), U?.140
- net PA2: now also U?.43 (PA2-LTDC_R1)
- net PA3: now also U?.46 (PA3-LTDC_B5)
- net PA4: now also U?.49 (PA4-DAC1_OUT1)
- net PA5: now also U?.50 (PA5-DAC1_OUT2)
- net PA6: now also U?.51 (PA6-OCTOSPIM_P1_IO3)
- net PA7: now also U?.52 (PA7-LTDC_VSYNC)
- net PA8: now also U?.127 (PA8-LTDC_B3)
- net PA9: now also U?.128 (PA9-LTDC_R5)
- net PB0: now also U?.55 (PB0-LTDC_R3)
- net PB1: now also U?.56 (PB1-LTDC_R6)
- net PB10: now also U?.78 (PB10-I2C2_SCL)
- net PB11: now also U?.79 (PB11-I2C2_SDA)
- net PB15: now also U?.88 (PB15-LTDC_G7)
- net PB2: now also U?.57 (PB2-OCTOSPIM_P1_CLK)
- net PB6: now also U?.165 (PB6-I2C1_SCL)
- net PB7: now also U?.166 (PB7-I2C1_SDA)
- net PC0: now also U?.34 (PC0-LTDC_G2)
- net PC1: now also U?.35 (PC1-LTDC_G5)
- net PC11: now also U?.141 (PC11-UART4_RX)
- net PC2_C: now also U?.36 (PC2_C-ADC3_INP0)
- net PC3_C: now also U?.37 (PC3_C-OCTOSPIM_P1_IO6)
- net PC4: now also U?.53 (PC4-LTDC_R7)
- net PC5: now also U?.54 (PC5-OCTOSPIM_P1_DQS)
- net PC6: now also U?.122 (PC6-LTDC_HSYNC)
- net PC9: now also U?.125 (PC9-LTDC_B2)
- net PD10: now also U?.91 (PD10-GPIO_Output)
- net PD2: now also U?.145 (PD2-LTDC_B7)
- net PDR_ON: now also R?.1, U?.174
- net PE10: now also U?.72 (PE10-OCTOSPIM_P1_IO7)
- net PE11: now also U?.73 (PE11-LTDC_G3)
- net PE12: now also U?.74 (PE12-LTDC_B4)
- net PE14: now also U?.76 (PE14-LTDC_CLK)
- net PE2: now also U?.1 (PE2-OCTOSPIM_P1_IO2)
- net PE4: now also U?.3 (PE4-LTDC_B0)
- net PE5: now also U?.4 (PE5-LTDC_G0)
- net PE6: now also U?.5 (PE6-LTDC_G1)
- net PE7: now also U?.67 (PE7-OCTOSPIM_P1_IO4)
- net PF0: now also U?.18 (PF0-OCTOSPIM_P2_IO0)
- net PF1: now also U?.19 (PF1-OCTOSPIM_P2_IO1)
- net PF10: now also U?.30 (PF10-LTDC_DE)
- net PF11: now also U?.58 (PF11-ADC1_INP2)
- net PF12: now also U?.59 (PF12-OCTOSPIM_P2_DQS)
- net PF13: now also U?.60 (PF13-ADC2_INP2)
- net PF14: now also U?.61 (PF14-I2C4_SCL)
- net PF15: now also U?.62 (PF15-I2C4_SDA)
- net PF2: now also U?.20 (PF2-OCTOSPIM_P2_IO2)
- net PF3: now also U?.21 (PF3-OCTOSPIM_P2_IO3)
- net PF4: now also U?.22 (PF4-OCTOSPIM_P2_CLK)
- net PF6: now also U?.26 (PF6-TIM23_CH1)
- net PF7: now also U?.27 (PF7-TIM23_CH2)
- net PF8: now also U?.28 (PF8-OCTOSPIM_P1_IO0)
- net PF9: now also U?.29 (PF9-OCTOSPIM_P1_IO1)
- net PG0: now also U?.63 (PG0-OCTOSPIM_P2_IO4)
- net PG1: now also U?.66 (PG1-OCTOSPIM_P2_IO5)
- net PG10: now also U?.154 (PG10-OCTOSPIM_P2_IO6)
- net PG11: now also U?.155 (PG11-OCTOSPIM_P2_IO7)
- net PG12: now also U?.156 (PG12-OCTOSPIM_P2_NCS)
- net PG13: now also U?.157 (PG13-LTDC_R0)
- net PG15: now also U?.161 (PG15-GPIO_Output)
- net PG2: now also U?.110 (PG2-GPIO_EXTI2)
- net PG3: now also U?.111 (PG3-GPIO_Output)
- net PG6: now also U?.116 (PG6-OCTOSPIM_P1_NCS)
- net PH0: now also U?.31 (PH0-OSC_IN-RCC_OSC_IN)
- net PJ11: now also U?.104 (PJ11-LTDC_G4)
- net PK1: now also U?.108 (PK1-LTDC_G6)
- net VDDSMPS: now also U?.16
- net VDD_SDC: now also C?.2, C?.2, U?.133, U?.135, U?.17, U?.172, U?.175, U?.80, U?.82
- net VLXSMPS: now also U?.15
- net VSSSMPS: now also U?.14
- net at JP1.3 (B): now also U?.39
- net at FB2.2: now also U?.40
- new net PB12: U?.85 (PB12-GPIO_Output)
- new net PB13: U?.86 (PB13-GPIO_Output)
- new net PC15: U?.139 (PA15(JTDI)-LTDC_B6)
- new net PD11: U?.94 (PD11-GPIO_Output)
- new net PD12: U?.95 (PD12-GPIO_Output)
- new net PD13: U?.96 (PD13-GPIO_Output)
- new net PD14: U?.97 (PD14-GPIO_Output)
- new net PD15: U?.98 (PD15-GPIO_Output)
- new net PE8: U?.68 (PE8-OCTOSPIM_P1_IO5)
Other:
- moved on the sheet: C14, J4

Commit message: more schematic work done: DAC output
Parts:
- removed U? (x2): STM32H735IGT6, Private:LQFP176_STM32H735IGT6_STM-M, symbol Private:STM32H735IGT6
- added C13, C14: 1nF, Capacitor_SMD:C_0805_2012Metric_Pad1.18x1.45mm_HandSolder, symbol Device:C
- added C18, C? (x4): 10uF, Capacitor_SMD:C_0805_2012Metric_Pad1.18x1.45mm_HandSolder, symbol Device:C
- added C19, C20: 100nF, Capacitor_SMD:C_0805_2012Metric_Pad1.18x1.45mm_HandSolder, symbol Device:C
- added J?: Conn_01x04_Socket, symbol Connector:Conn_01x04_Socket
- added JP? (x2): SolderJumper_3_Open, Jumper:SolderJumper-3_P1.3mm_Open_Pad1.0x1.5mm_NumberLabels, symbol Jumper:SolderJumper_3_Open
- added R10, R11, R4, R5, R6, R7, R8, R9: 10k, Resistor_SMD:R_0805_2012Metric_Pad1.20x1.40mm_HandSolder, symbol Device:R
- added U2: STM32H735IGT6, Private:LQFP176_STM32H735IGT6_STM-M, symbol Private:STM32H735IGT6
- added U? (x3): OPA1678IDGKT, Private:OPA1678_L, symbol Private:OPA1678IDGKT
- gave numbers to parts that had none: 4
- renumbered C14 to C16, R4 to R12, R5 to R13, R6 to R14, R7 to R15, R8 to R16, R9 to R17, R12 to R18, R13 to R19, R14 to R20
Connections:
- net SCL1 is gone; now on net PB6: JI2C3.3 (Pin_3), R17.1
- net SCL2 is gone; now on net PB10: JI2C2.3 (Pin_3), R16.1
- net SCL4 is gone; now on net PF14: JI2C1.3 (Pin_3), R15.1
- net SDA1 is gone; now on net PB7: JI2C3.2 (Pin_2), R14.1
- net SDA2 is gone; now on net PB11: JI2C2.2 (Pin_2), R13.1
- net SDA4 is gone; now on net PF15: JI2C1.2 (Pin_2), R12.1
- net UART_RX is gone; now on net PC11: JUART1.2 (Pin_2)
- net UART_TX is gone; now on net PA0: JUART1.3 (Pin_3)
- net +3.3V: now also J4.45, J4.50, C18.1, C19.1, C20.1, J?.2 (Pin_2), U2.105, U2.113, U2.126, U2.13, U2.136, U2.152, U2.160, U2.176, U2.25, U2.44, U2.48, U2.65, U2.7, U2.71, U2.8, U2.84, U2.92, U2.99
- net +5V: now also J?.3 (Pin_3), JP?.3 (B), JP?.3 (B), U?.8 (V+)
- net BOOT0: now also U2.167
- net GND: now also J4.1, J4.19, J4.2, J4.20, J4.30, J4.34, J4.37, J4.47, J4.49, C18.2, C19.2, C20.2, J?.1 (Pin_1), R8.1, R9.1, U2.100, U2.106, U2.112, U2.119, U2.12, U2.121, U2.134, U2.137, U2.151, U2.159, U2.173, U2.24, U2.38, U2.45, U2.47, U2.6, U2.64, U2.70, U2.81, U2.83, U2.93
- net NRST: now also J4.36, U2.33
- net PA0: now also U2.41 (PA0-UART4_TX)
- net PA1: now also U2.42 (PA1-LTDC_R2)
- net PA10: now also U2.129 (PA10-LTDC_B1)
- net PA11: now also U2.130 (PA11-LTDC_R4)
- net PA13: now also U2.132 (PA13(JTMS/SWDIO)-DEBUG_JTMS-SWDIO)
- net PA14: now also U2.138 (PA14(JTCK/SWCLK)-DEBUG_JTCK-SWCLK), U2.140
- net PA2: now also U2.43 (PA2-LTDC_R1)
- net PA3: now also U2.46 (PA3-LTDC_B5)
- net PA4: now also C?.1, U2.49 (PA4-DAC1_OUT1)
- net PA5: now also C?.1, U2.50 (PA5-DAC1_OUT2)
- net PA6: now also U2.51 (PA6-OCTOSPIM_P1_IO3)
- net PA7: now also U2.52 (PA7-LTDC_VSYNC)
- net PA8: now also J4.27, U2.127 (PA8-LTDC_B3)
- net PA9: now also U2.128 (PA9-LTDC_R5)
- net PB0: now also U2.55 (PB0-LTDC_R3)
- net PB1: now also U2.56 (PB1-LTDC_R6)
- net PB10: now also U2.78 (PB10-I2C2_SCL)
- net PB11: now also U2.79 (PB11-I2C2_SDA)
- net PB12: now also U2.85 (PB12-GPIO_Output)
- net PB13: now also U2.86 (PB13-GPIO_Output)
- net PB15: now also U2.88 (PB15-LTDC_G7)
- net PB2: now also U2.57 (PB2-OCTOSPIM_P1_CLK)
- net PB6: now also U2.165 (PB6-I2C1_SCL)
- net PB7: now also U2.166 (PB7-I2C1_SDA)
- net PC0: now also U2.34 (PC0-LTDC_G2)
- net PC1: now also U2.35 (PC1-LTDC_G5)
- net PC11: now also U2.141 (PC11-UART4_RX)
- net PC15: now also U2.139 (PA15(JTDI)-LTDC_B6)
- net PC2_C: now also U2.36 (PC2_C-ADC3_INP0)
- net PC3_C: now also U2.37 (PC3_C-OCTOSPIM_P1_IO6)
- net PC4: now also U2.53 (PC4-LTDC_R7)
- net PC5: now also U2.54 (PC5-OCTOSPIM_P1_DQS)
- net PC6: now also U2.122 (PC6-LTDC_HSYNC)
- net PC9: now also U2.125 (PC9-LTDC_B2)
- net PD10: now also J4.24, U2.91 (PD10-GPIO_Output); no longer J4.27
- net PD11: now also U2.94 (PD11-GPIO_Output)
- net PD12: now also U2.95 (PD12-GPIO_Output)
- net PD13: now also U2.96 (PD13-GPIO_Output)
- net PD14: now also U2.97 (PD14-GPIO_Output)
- net PD15: now also U2.98 (PD15-GPIO_Output)
- net PD2: now also U2.145 (PD2-LTDC_B7)
- net PDR_ON: now also U2.174
- net PE10: now also U2.72 (PE10-OCTOSPIM_P1_IO7)
- net PE11: now also U2.73 (PE11-LTDC_G3)
- net PE12: now also U2.74 (PE12-LTDC_B4)
- net PE14: now also J4.32, U2.76 (PE14-LTDC_CLK); no longer J4.30
- net PE2: now also U2.1 (PE2-OCTOSPIM_P1_IO2)
- net PE4: now also U2.3 (PE4-LTDC_B0)
- net PE5: now also U2.4 (PE5-LTDC_G0)
- net PE6: now also U2.5 (PE6-LTDC_G1)
- net PE7: now also U2.67 (PE7-OCTOSPIM_P1_IO4)
- net PE8: now also U2.68 (PE8-OCTOSPIM_P1_IO5)
- net PF0: now also U2.18 (PF0-OCTOSPIM_P2_IO0)
- net PF1: now also U2.19 (PF1-OCTOSPIM_P2_IO1)
- net PF10: now also U2.30 (PF10-LTDC_DE)
- net PF11: now also U2.58 (PF11-ADC1_INP2)
- net PF12: now also U2.59 (PF12-OCTOSPIM_P2_DQS)
- net PF13: now also U2.60 (PF13-ADC2_INP2)
- net PF14: now also U2.61 (PF14-I2C4_SCL)
- net PF15: now also U2.62 (PF15-I2C4_SDA)
- net PF2: now also U2.20 (PF2-OCTOSPIM_P2_IO2)
- net PF3: now also U2.21 (PF3-OCTOSPIM_P2_IO3)
- net PF4: now also U2.22 (PF4-OCTOSPIM_P2_CLK)
- net PF6: now also U2.26 (PF6-TIM23_CH1)
- net PF7: now also U2.27 (PF7-TIM23_CH2)
- net PF8: now also U2.28 (PF8-OCTOSPIM_P1_IO0)
- net PF9: now also U2.29 (PF9-OCTOSPIM_P1_IO1)
- net PG0: now also U2.63 (PG0-OCTOSPIM_P2_IO4)
- net PG1: now also U2.66 (PG1-OCTOSPIM_P2_IO5)
- net PG10: now also U2.154 (PG10-OCTOSPIM_P2_IO6)
- net PG11: now also U2.155 (PG11-OCTOSPIM_P2_IO7)
- net PG12: now also U2.156 (PG12-OCTOSPIM_P2_NCS)
- net PG13: now also U2.157 (PG13-LTDC_R0)
- net PG15: now also U2.161 (PG15-GPIO_Output)
- net PG2: now also U2.110 (PG2-GPIO_EXTI2)
- net PG3: now also U2.111 (PG3-GPIO_Output); no longer J4.24
- net PG6: now also U2.116 (PG6-OCTOSPIM_P1_NCS)
- net PH0: now also U2.31 (PH0-OSC_IN-RCC_OSC_IN)
- net PJ11: now also U2.104 (PJ11-LTDC_G4)
- net PK1: now also U2.108 (PK1-LTDC_G6)
- net VDDSMPS: now also U2.16
- net VDD_SDC: now also U2.133, U2.135, U2.17, U2.172, U2.175, U2.80, U2.82
- net VLXSMPS: now also U2.15
- net VSSSMPS: now also U2.14
- net at JP1.3 (B): now also U2.39
- net at FB2.2: now also U2.40
- net DAC1: no longer names the net of JDAC1.2 (Pin_2)
- net DAC1: now also C?.2
- net DAC2: no longer names the net of JDAC1.3 (Pin_3)
- net DAC2: now also C?.2
- new net: R7.1, R9.2, U?.5 (IN+)
- new net: JP?.2 (C), R7.2
- new net: R6.1, R8.2, U?.3 (IN+)
- new net: JP?.2 (C), R6.2
- new net: C?.2, R5.2
- new net: C14.2, C?.1, R11.1, U?.7 (OUT)
- new net: C14.1, R11.2, R5.1, U?.6 (IN-)
- new net: C13.2, C?.1, R10.1, U?.1 (OUT)
- new net: C13.1, R10.2, R4.1, U?.2 (IN-)
- new net: C?.2, R4.2
- new net -5V: J?.4 (Pin_4), JP?.1 (A), JP?.1 (A), U?.4 (V-)
- no-connect marks 12 -> 17
Other:
- note added: "ADC3: 2: INP0 PC2_C"
- note added: "DAC1: 2: OUT1 PA4 3: OUT2 PA5"
- note added: "I2C1: 2: SDA PB7 3: SCL PB6"
- note added: "I2C2: 2: SDA PB11 3: SCL PB10"
- note added: "I2C4: 2: SDA PF15 3: SCL PF14"
- note added: "UART4: 2: RX PC11 3: TX PA0"
- note added: "all I2C pull-up resistors: 3x2 4.7k"
- note added: "package size / footprint?"
- moved on the sheet: R22

Commit message: more KiCAD work performed
Parts:
- added C21, C22, C23: PGB1010603, Capacitor_SMD:C_0603_1608Metric, symbol Private:PGB1010603
- added JGPIO1: Conn_01x03_Socket, Connector_JST:JST_XH_B3B-XH-A_1x03_P2.50mm_Vertical, symbol Connector:Conn_01x03_Socket
- added R3: 10k, Resistor_SMD:R_0805_2012Metric_Pad1.20x1.40mm_HandSolder, symbol Device:R
- C1: footprint PGB1010603:ESD_PGB1010603MR -> Capacitor_SMD:C_0603_1608Metric
- J1: renamed from J?; footprint (none) -> Connector_JST:JST_XH_B4B-XH-A_1x04_P2.50mm_Vertical
- gave numbers to parts that had none: 7
- renumbered C10 to C12, C11 to C13, C13 to C14, C14 to C15, C12 to C16, C15 to C19, C16 to C20, C17 to C24, C18 to C25, C19 to C26, C20 to C27, J1 to J2, JP1 to JP3, J2 to JRadio1, R9 to R10, R10 to R11, R11 to R12, R12 to R13, R13 to R14, R14 to R15, R15 to R16, R16 to R17, R17 to R18, R18 to R19, R19 to R20, R20 to R21, R21 to R22, R22 to R23, R3 to R4, R4 to R5, R5 to R6, R6 to R7, R7 to R8, R8 to R9
Connections:
- net ADC1 is gone; now on net PF11: JRadio1.19 (Pin_19)
- net ADC2 is gone; now on net PF13: JRadio1.20 (Pin_20)
- net LSBUSB is gone; now on net PD13: JRadio1.11 (Pin_11), JRadio1.12 (Pin_12)
- net RXTX is gone; now on net PD15: JRadio1.3 (Pin_3), JRadio1.4 (Pin_4), JRadio1.5 (Pin_5), JRadio1.6 (Pin_6)
- net R_CH1 is gone; now on net PF6: JRadio1.17 (Pin_17)
- net R_CH2 is gone; now on net PF7: JRadio1.18 (Pin_18)
- net S0 is gone; now on net PD12: JRadio1.13 (Pin_13), JRadio1.14 (Pin_14)
- net S1 is gone; now on net PD11: JRadio1.15 (Pin_15), JRadio1.16 (Pin_16)
- net nRXTX is gone; now on net PD14: JRadio1.10 (Pin_10), JRadio1.7 (Pin_7), JRadio1.8 (Pin_8), JRadio1.9 (Pin_9)
- net +3.3V: now also R3.1
- net GND: now also H1.MP, H2.MP, H3.MP, H4.MP, H5.MP, H6.MP, H7.MP, H8.MP, C21.2, C22.1, C23.1, JGPIO1.1 (Pin_1)
- net PB12: now also JGPIO1.2 (Pin_2)
- net PB13: now also JGPIO1.3 (Pin_3)
- net PC2_C: no longer UFLASH1.E3 (SIO5)
- net PE8: now also UFLASH1.E3 (SIO5)
- net PG6: no longer UFLASH1.A5 (~{ECS})
- net at J3.2, R19.2: now also C21.1
- net at J3.4, R20.2: now also C22.2
- net at J3.10, R21.2: now also C23.2
- new net: R3.2, UFLASH1.A5 (~{ECS})
Other:
- note added: "Radio Connectors: RXTX: PD15 NRXTX: PD14 LSBUSB: PD13 S0: PD12 S1: PD11 TIM23_CH1: PF6 TIM23_CH2: PF7 ADC1_INP2: PF11 ADC2_INP2: PF13"
- note added: "do not fit"
- moved on the sheet: H5, H6, H7, H8, R19, R20, R21

Commit message: finished schematics, check with AS performed
Parts:
- removed H1, H2, H3, H4, H5, H6, H7, H8: MountingHole_Pad_MP, MountingHole:MountingHole_2.7mm_M2.5_Pad_TopBottom, symbol Mechanical:MountingHole_Pad_MP
- removed J1: Conn_01x04_Socket, Connector_JST:JST_XH_B4B-XH-A_1x04_P2.50mm_Vertical, symbol Connector:Conn_01x04_Socket
- added C1, C6: 47uF Tant. 25V, Capacitor_Tantalum_SMD:CP_EIA-7343-30_AVX-N_Pad2.25x2.55mm_HandSolder, symbol Device:C_Polarized_Small
- added C13: 100uF Tant. 25V, Capacitor_Tantalum_SMD:CP_EIA-7343-30_AVX-N_Pad2.25x2.55mm_HandSolder, symbol Device:C_Polarized_Small
- added C15: 1uF, Capacitor_SMD:C_0805_2012Metric_Pad1.18x1.45mm_HandSolder, symbol Device:C_Small
- added C17, C3, C5: 100nF, Capacitor_SMD:C_0805_2012Metric_Pad1.18x1.45mm_HandSolder, symbol Device:C_Small
- added C19, C2: 10uF Tant. 25V, Capacitor_Tantalum_SMD:CP_EIA-7343-30_AVX-N_Pad2.25x2.55mm_HandSolder, symbol Device:C_Polarized_Small
- added C4: optional: 82pF, Capacitor_SMD:C_0805_2012Metric_Pad1.18x1.45mm_HandSolder, symbol Device:C_Small
- added C7: 1uF, Tant. 25V, Capacitor_Tantalum_SMD:CP_EIA-7343-30_AVX-N_Pad2.25x2.55mm_HandSolder, symbol Device:C_Polarized_Small
- added D1: PMEG2010AEH, Diode_SMD:D_SOD-123F, symbol Diode:PMEG2010AEH
- added H1, H2, H3, H4: MountingHole_Pad, MountingHole:MountingHole_3.2mm_M3_Pad_TopBottom, symbol Mechanical:MountingHole_Pad
- added IC1: NCP700BSN33T1G, Private:SOT95P275X120-5N, symbol Private:NCP700BSN33T1G
- added JPOWER1: Conn_01x02_Socket, Connector_JST:JST_XH_B2B-XH-A_1x02_P2.50mm_Vertical, symbol Connector:Conn_01x02_Socket
- added L1: 10uH, Inductor_SMD:L_1812_4532Metric_Pad1.30x3.40mm_HandSolder, symbol Device:L
- added PS1: TPS6735ID, Private:SOIC127P600X175-8N, symbol Private:TPS6735ID
- added U1: L7805, Package_TO_SOT_THT:TO-220-3_Horizontal_TabDown, symbol Regulator_Linear:L7805
- J1: renamed from J2; footprint Connector_JST:JST_XH_B2B-XH-AM_1x02_P2.50mm_Vertical -> Connector_JST:JST_XH_B3B-XH-A_1x03_P2.50mm_Vertical
- JADC1: footprint Connector_JST:JST_XH_B3B-XH-A_1x03_P2.50mm_Vertical -> Connector_JST:JST_XH_B2B-XH-A_1x02_P2.50mm_Vertical
- renumbered C3 to C10, C4 to C11, C5 to C12, C6 to C14, C7 to C16, C8 to C18, C9 to C20, C10 to C21, C11 to C22, C12 to C23, C13 to C24, C14 to C25, C15 to C26, C16 to C27, C17 to C28, C18 to C29, C19 to C30, C20 to C31, C21 to C32, C22 to C33, C23 to C34, C24 to C35, C25 to C36, C26 to C37, C27 to C38, C1 to C8, C2 to C9, J3 to J2, J4 to J3, L1 to L2, U1 to U2, U2 to U3
Connections:
- net PC15 is gone; now on net PA15: U3.139 (PA15(JTDI)-LTDC_B6)
- net +3.3V: now also C17.1, C19.1, IC1.5 (OUT); no longer C11.1, C16.1, C20.1, C36.1, C37.1, FB1.1, J3.45, JP3.1 (A), U3.105, U3.113, U3.126, U3.13, U3.136, U3.152, U3.160, U3.176, U3.25, U3.44, U3.48, U3.65, U3.7, U3.71, U3.8, U3.84, U3.92, U3.99, UHYPERRAM1.B4 (VCC), UHYPERRAM1.D1 (VCCQ), UHYPERRAM1.E4 (VCCQ)
- net +5V: now also C36.1, C37.1, J3.45, C5.1, C6.1, C7.1, IC1.1 (IN), IC1.3 (EN), PS1.1 (EN), PS1.8 (VCC), U1.3 (OUT)
- net -5V: now also C13.2, D1.2 (A), PS1.5 (FB)
- net GND: now also C1.2, C13.1, C15.1, C17.2, C19.2, C2.2, C3.2, C4.2, C5.2, C6.2, C7.2, H1.1, H2.1, H3.1, H4.1, IC1.2 (GND), JPOWER1.1 (Pin_1), L1.2, PS1.6 (GND), U1.2 (GND); no longer U3.100, U3.106, U3.112, U3.119, U3.12, U3.121, U3.134, U3.137, U3.151, U3.159, U3.173, U3.24, U3.38, U3.45, U3.47, U3.6, U3.64, U3.70, U3.81, U3.83, U3.93, UHYPERRAM1.B3 (VSS), UHYPERRAM1.C1 (VSSQ), UHYPERRAM1.E5 (VSSQ)
- new net: C2.1, PS1.2 (REF)
- new net: C1.1, C3.1, JPOWER1.2 (Pin_2), U1.1 (IN)
- new net: C4.1, PS1.4 (COMP)
- new net: D1.1 (K), L1.1, PS1.7 (OUT)
- new net: C15.2, IC1.4 (BYP)
- new net VDD: C11.1, C16.1, C20.1, FB1.1, JP3.1 (A), U3.105, U3.113, U3.126, U3.13, U3.136, U3.152, U3.160, U3.176, U3.25, U3.44, U3.48, U3.65, U3.7, U3.71, U3.8, U3.84, U3.92, U3.99, UHYPERRAM1.B4 (VCC), UHYPERRAM1.D1 (VCCQ), UHYPERRAM1.E4 (VCCQ)
- new net VSS: U3.100, U3.106, U3.112, U3.119, U3.12, U3.121, U3.134, U3.137, U3.151, U3.159, U3.173, U3.24, U3.38, U3.45, U3.47, U3.6, U3.64, U3.70, U3.81, U3.83, U3.93, UHYPERRAM1.B3 (VSS), UHYPERRAM1.C1 (VSSQ), UHYPERRAM1.E5 (VSSQ)
- no-connect marks 17 -> 18
