File: CustomSTM32H735Board/KiCADFiles/CustomSTM32H735_V2_Board/CustomSTM32H735_V2_Board/CustomSTM32H735_V2_Board.kicad_sch (KiCad schematic)
At the start: 99 parts, among them IC1 NCP700BSN33T1G, J1 FLE-125-01-G-DV, SW1 SW_Omron_B3FS, U1 L7805, U2 OPA1678IDGKT, U3 STM32H735IGT6, X1 NSC5004A-25M

Commit message: KiCAD V2 board progress
Parts:
- removed R22: 5k1, Resistor_SMD:R_0805_2012Metric_Pad1.20x1.40mm_HandSolder, symbol Device:R
- removed TP5: TestPoint, Connector_Pin:Pin_D0.7mm_L6.5mm_W1.8mm_FlatFork, symbol Connector:TestPoint
- removed U3: STM32H735IGT6, Private:LQFP176_STM32H735IGT6_STM-M, symbol Private:STM32H735IGT6
- added R?: 5k1, Resistor_SMD:R_0805_2012Metric_Pad1.20x1.40mm_HandSolder, symbol Device:R
- added TP?: TestPoint, Connector_Pin:Pin_D0.7mm_L6.5mm_W1.8mm_FlatFork, symbol Connector:TestPoint
- added U? (x3): STM32H735IGK6, Private:BGA_735IGK6_STM, symbol Private:STM32H735IGK6
Connections:
- net PA10 is gone; now on net PD0: J1.23
- net PA7 is gone; now on net PA4: J1.28
- net PC0 is gone; now on net PA6: J1.8
- net PE5 is gone; now on net PB1: J1.4
- net PE6 is gone; now on net PB0: J1.6
- net PF8 is gone; now on net PD11: UFLASH1.D3 (SI/SIO0)
- net PF9 is gone; now on net PD12: UFLASH1.D2 (SO/SIO1)
- net +3.3V: now also U?.D11 (VDD), U?.D5 (VDD), U?.E12 (VDD), U?.E4 (VDD), U?.G4 (VDD), U?.H12 (VDD), U?.K4 (VDD), U?.L12 (VDD), U?.M5 (VDD), U?.M9 (VDD)
- net BOOT0: now also R?.1, U?.C5 (BOOT0)
- net GND: now also R?.2, U?.A1 (VSS), U?.C2 (VSS), U?.D10 (VSS), U?.D6 (VSS), U?.E1 (VSS), U?.F10 (VSS), U?.F12 (VSS), U?.F6 (VSS), U?.F7 (VSS), U?.F8 (VSS), U?.F9 (VSS), U?.G10 (VSS), U?.G6 (VSS), U?.G7 (VSS), U?.G8 (VSS), U?.G9 (VSS), U?.H10 (VSS), U?.H6 (VSS), U?.H7 (VSS), U?.H8 (VSS), U?.H9 (VSS), U?.J10 (VSS), U?.J14 (VSS), U?.J6 (VSS), U?.J7 (VSS), U?.J8 (VSS), U?.J9 (VSS), U?.K10 (VSS), U?.K12 (VSS), U?.K2 (VSS), U?.K6 (VSS), U?.K7 (VSS), U?.K8 (VSS), U?.K9 (VSS), U?.M10 (VSS), U?.M6 (VSS), U?.R15 (VSS)
- net NRST: now also TP?.1, U?.L1 (NRST)
- net PA0: now also U?.P1 (PA0-VSYNC_FREQ), U?.R3 (PA0_C-ADC1_INP0)
- net PA13: now also U?.B13 (PA13(JTMS/SWDIO)-DEBUG_JTMS-SWDIO)
- net PA14: now also U?.A12 (PA14(JTCK/SWCLK)-DEBUG_JTCK-SWCLK)
- net PA15: now also U?.A11 (PA15(JTDI)-TIM2_CH1); no longer J1.33
- net PA3: now also U?.N5 (PA3-LTDC_B5)
- net PA4: now also U?.P5 (PA4-LTDC_VSYNC)
- net PA5: now also U?.P6 (PA5-DAC1_OUT2)
- net PA6: now also U?.R7 (PA6-LTDC_G2); no longer UFLASH1.D4 (SIO3)
- net PA8: now also U?.B14 (PA8-LTDC_B3)
- net PB0: now also U?.R8 (PB0-LTDC_G1); no longer J1.9
- net PB1: now also U?.M8 (PB1-LTDC_G0); no longer J1.15
- net PB10: now also U?.N12 (PB10-I2C2_SCL)
- net PB11: now also U?.P10 (PB11-I2C2_SDA)
- net PB12: now also U?.M15 (PB12-S0)
- net PB13: now also U?.L15 (PB13-S1)
- net PB15: now also U?.K14 (PB15-MCU_ACTIVE), U?.K15 (PB14-FRAME_RATE); no longer J1.18
- net PB2: now also UFLASH1.C3 (DQS); no longer UFLASH1.B2 (SCLK)
- net PB6: now also U?.A5 (PB6-OCTOSPIM_P1_NCS)
- net PC2_C: now also U?.N1 (PC2_C-ADC3_INP0)
- net PC4: now also U?.R6 (PC4-OPAMP1_VOUT); no longer J1.17
- net PC5: now also U?.M7 (PC5-OCTOSPIM_P1_DQS); no longer UFLASH1.C3 (DQS)
- net PC6: now also U?.E14 (PC6-LTDC_HSYNC)
- net PC9: now also U?.E13 (PC9-OCTOSPIM_P1_IO0); no longer J1.25
- net PD0: now also U?.C10 (PD0-LTDC_B1); no longer JP4.3 (B)
- net PD10: now also U?.L13 (PD10-LCD_DISP)
- net PD12: now also U?.J15 (PD12-LSBUSB)
- net PD13: now also UFLASH1.D4 (SIO3), U?.H15 (PD13-GPIOPD13)
- net PE11: now also U?.R12 (PE11-LTDC_G3)
- net PE12: now also U?.P12 (PE12-LTDC_B4)
- net PE2: now also U?.C3 (PE2-OCTOSPIM_P1_IO2)
- net PF0: now also U?.F4 (PF0-OCTOSPIM_P2_IO0)
- net PF1: now also U?.F3 (PF1-OCTOSPIM_P2_IO1)
- net PF10: now also UFLASH1.B2 (SCLK), U?.K3 (PF10-OCTOSPIM_P1_CLK); no longer J1.22
- net PF11: now also U?.N7 (PF11-TIM24_CH1)
- net PF12: now also U?.P11 (PF12-TIM24_CH2)
- net PF2: now also U?.G3 (PF2-OCTOSPIM_P2_IO2)
- net PF3: now also U?.H4 (PF3-OCTOSPIM_P2_IO3)
- net PF4: now also U?.H2 (PF4-OCTOSPIM_P2_CLK)
- net PF6: now also U?.H1 (PF6-OCTOSPIM_P1_IO3)
- net PG0: now also U?.P8 (PG0-OCTOSPIM_P2_IO4)
- net PG1: now also U?.N9 (PG1-OCTOSPIM_P2_IO5)
- net PG10: now also U?.C8 (PG10-OCTOSPIM_P2_IO6)
- net PG11: now also U?.A7 (PG11-OCTOSPIM_P2_IO7)
- net PG12: now also U?.D8 (PG12-OCTOSPIM_P2_NCS)
- net PG15: now also U?.D7 (PG15-OCTOSPIM_P2_DQS)
- net PG3: now also U?.H13 (PG3-RENDER_TIME)
- net PH0: now also U?.J1 (PH0-OSC_IN-RCC_OSC_IN)
- net PA1 renamed PH8
- net PH8: now also U?.N13 (PH8-LTDC_R2)
- net PA11 renamed PH10
- net PH10: now also U?.N14 (PH10-LTDC_R4)
- net PA2 renamed PH3
- net PH3: now also U?.R4 (PH3-LTDC_R1)
- net PA9 renamed PH11
- net PH11: now also U?.M13 (PH11-LTDC_R5)
- net PC1 renamed PH4
- net PH4: now also U?.P4 (PH4-LTDC_G5)
- net PC3_C renamed PG9
- net PG9: now also U?.A8 (PG9-OCTOSPIM_P1_IO6)
- net PD2 renamed PB9
- net PB9: now also U?.B3 (PB9-LTDC_B7)
- net PE10 renamed PED7
- net PE14 renamed ??
- net PE4 renamed PG14
- net PG14: now also U?.C7 (PG14-LTDC_B0)
- net PE7 renamed PD4
- net PD4: now also U?.C9 (PD4-OCTOSPIM_P1_IO4)
- net PE8 renamed PD5
- net PD5: now also U?.B9 (PD5-OCTOSPIM_P1_IO5)
- net PG13 renamed PE0
- net PE0: now also U?.B4 (PE0-LTDC_R0)
- net PJ11 renamed PH15
- net PH15: now also U?.D12 (PH15-LTDC_G4)
- net PK1 renamed PC7
- net PC7: now also U?.D15 (PC7-LTDC_G6)
- new net P??: JP4.3 (B)
- new net PB3: U?.A6 (PB3(JTDO/TRACESWO)-TIM2_CH2)
- new net PB8: J1.33, U?.A2 (PB8-LTDC_B6)
- new net PC10: U?.C12 (PC10-OCTOSPIM_P1_IO1)
- new net PD1: U?.A10 (PD1-UART4_TX)
- new net PD3: J1.18, U?.A9 (PD3-LTDC_G7)
- new net PD6: J1.25, U?.D9 (PD6-LTDC_B2)
- new net PD7: U?.B8 (PD7-OCTOSPIM_P1_IO7)
- new net PE1: J1.15, U?.C4 (PE1-LTDC_R6)
- new net PE13: J1.22, U?.P13 (PE13-LTDC_DE)
- new net PE15: J1.17, U?.P14 (PE15-LTDC_R7)
- new net PG7: U?.G13 (PG7-LTDC_CLK)
- new net PH12: U?.N15 (PH12-NRXTX)
- new net PH14: U?.B12 (PH14-UART4_RX)
- new net PH6: U?.P15 (PH6-RXTX)
- new net PH9: J1.9, U?.M14 (PH9-LTDC_R3)
- no-connect marks 58 -> 38
Other:
- moved on the sheet: C10, C11, C12, C14, C16, C18, C20, C23, C24, C27, C30, C31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
