File: CustomSTM32H735Board/KiCADFiles/CustomSTM32H735_V2_Board/CustomSTM32H735_V2_Board/CustomSTM32H735_V2_Board.kicad_sch (KiCad schematic)
At the start: 101 parts, among them IC1 NCP700BSN33T1G, J1 FLE-125-01-G-DV, SW1 SW_Omron_B3FS, U1 L7805, U2 OPA1678IDGKT, X1 NSC5004A-25M

Commit message: board schematics V2 checked and final
Parts:
- removed C30, C31, C35: 4.7uF low ESR, Capacitor_SMD:C_0805_2012Metric_Pad1.18x1.45mm_HandSolder, symbol Device:C
- removed R23: 1k, Resistor_SMD:R_0805_2012Metric_Pad1.20x1.40mm_HandSolder, symbol Device:R
- removed U? (x3): STM32H735IGK6, Private:BGA_735IGK6_STM, symbol Private:STM32H735IGK6
- added C18, C34, C38: 4.7uF low ESR, Capacitor_SMD:C_0805_2012Metric_Pad1.18x1.45mm_HandSolder, symbol Device:C
- added JFRAME1: Conn_01x04_Socket, symbol Connector:Conn_01x04_Socket
- added JTIM1: Conn_01x03_Socket, Connector_JST:JST_XH_B3B-XH-A_1x03_P2.50mm_Vertical, symbol Connector:Conn_01x03_Socket
- added R24: 0R, Resistor_SMD:R_0805_2012Metric_Pad1.20x1.40mm_HandSolder, symbol Device:R
- added R6: 10k, Resistor_SMD:R_0805_2012Metric_Pad1.20x1.40mm_HandSolder, symbol Device:R
- added TP_OSC_: TestPoint, Connector_Pin:Pin_D0.7mm_L6.5mm_W1.8mm_FlatFork, symbol Connector:TestPoint
- added U3: STM32H735IGK6, Private:BGA_735IGK6_STM, symbol Private:STM32H735IGK6
- U1: footprint Package_TO_SOT_THT:TO-220-3_Horizontal_TabDown -> Private:TO-220-3_Horizontal_TabDown_GND_Pad
- gave numbers to parts that had none: 2
- renumbered C8 to C1, C14 to C10, C16 to C11, C18 to C12, C5 to C13, C20 to C14, C6 to C15, C7 to C16, C13 to C17, C15 to C19, C9 to C2, C17 to C20, C19 to C21, C21 to C22, C22 to C23, C25 to C24, C26 to C25, C28 to C26, C29 to C27, C27 to C28, C24 to C29, C1 to C3, C23 to C30, C32 to C31, C33 to C32, C34 to C33, C36 to C35, C37 to C36, C38 to C37, C2 to C4, C3 to C5, C4 to C6, C10 to C7, C11 to C8, C12 to C9, R8 to R10, R9 to R11, R10 to R12, R11 to R13, R12 to R14, R13 to R15, R14 to R16, R15 to R17, R16 to R18, R17 to R19, R18 to R20, R19 to R21, R20 to R22, R21 to R23, R5 to R7, R6 to R8, R7 to R9, TP4 to TP_VDD_SDC_
Connections:
- net P?? is gone; now on net PH6: JP4.3 (B)
- net PB6 is gone; now on net PB10: JI2C3.3 (Pin_3), R20.1
- net PB7 is gone; now on net PB11: JI2C3.2 (Pin_2), R17.1
- net PC11 is gone; now on net PH14: JUART1.2 (Pin_2)
- net PD14 is gone; now on net PH12: JRadio1.10 (Pin_10), JRadio1.7 (Pin_7), JRadio1.8 (Pin_8), JRadio1.9 (Pin_9)
- net PED7 is gone; now on net PD7: UFLASH1.E1 (SIO7)
- net +3.3V: now also R6.2, U3.D11 (VDD), U3.D5 (VDD), U3.E12 (VDD), U3.E4 (VDD), U3.G4 (VDD), U3.H12 (VDD), U3.K4 (VDD), U3.L12 (VDD), U3.M5 (VDD), U3.M9 (VDD)
- net BOOT0: now also U3.C5 (BOOT0)
- net GND: now also C18.1, C34.1, C38.1, JTIM1.1 (Pin_1), U3.A1 (VSS), U3.A15 (VSS), U3.C2 (VSS), U3.D10 (VSS), U3.D6 (VSS), U3.E1 (VSS), U3.F10 (VSS), U3.F12 (VSS), U3.F2 (VSSSMPS), U3.F6 (VSS), U3.F7 (VSS), U3.F8 (VSS), U3.F9 (VSS), U3.G10 (VSS), U3.G6 (VSS), U3.G7 (VSS), U3.G8 (VSS), U3.G9 (VSS), U3.H10 (VSS), U3.H6 (VSS), U3.H7 (VSS), U3.H8 (VSS), U3.H9 (VSS), U3.J10 (VSS), U3.J14 (VSS), U3.J6 (VSS), U3.J7 (VSS), U3.J8 (VSS), U3.J9 (VSS), U3.K10 (VSS), U3.K12 (VSS), U3.K2 (VSS), U3.K6 (VSS), U3.K7 (VSS), U3.K8 (VSS), U3.K9 (VSS), U3.L4 (VREF-), U3.M10 (VSS), U3.M6 (VSS), U3.N3 (VSSA), U3.R1 (VSS), U3.R15 (VSS)
- net NRST: now also U3.L1 (NRST)
- net PA0: now also JFRAME1.4 (Pin_4), U3.P1 (PA0-VSYNC_FREQ); no longer JUART1.3 (Pin_3)
- net PA13: now also U3.B13 (PA13(JTMS/SWDIO)-DEBUG_JTMS-SWDIO)
- net PA14: now also U3.A12 (PA14(JTCK/SWCLK)-DEBUG_JTCK-SWCLK)
- net PA15: now also JTIM1.2 (Pin_2), U3.A11 (PA15(JTDI)-TIM2_CH1)
- net PA3: now also U3.N5 (PA3-LTDC_B5)
- net PA4: now also U3.P5 (PA4-LTDC_VSYNC); no longer C22.1
- net PA5: now also U3.P6 (PA5-DAC1_OUT2)
- net PA6: now also U3.R7 (PA6-LTDC_G2)
- net PA8: now also U3.B14 (PA8-LTDC_B3)
- net PB0: now also U3.R8 (PB0-LTDC_G1)
- net PB1: now also U3.M8 (PB1-LTDC_G0)
- net PB10: now also U3.N12 (PB10-I2C2_SCL); no longer JI2C2.3 (Pin_3), R19.1
- net PB11: now also U3.P10 (PB11-I2C2_SDA); no longer JI2C2.2 (Pin_2), R16.1
- net PB12: now also JRadio1.13 (Pin_13), JRadio1.15 (Pin_15), U3.M15 (PB12-S0); no longer JGPIO1.2 (Pin_2)
- net PB13: now also JRadio1.14 (Pin_14), JRadio1.16 (Pin_16), U3.L15 (PB13-S1); no longer JGPIO1.3 (Pin_3)
- net PB15: now also JFRAME1.2 (Pin_2), U3.K14 (PB15-MCU_ACTIVE)
- net PB2: now also U3.P7 (PB2-OCTOSPIM_P1_DQS)
- net PB3: now also JTIM1.3 (Pin_3), U3.A6 (PB3(JTDO/TRACESWO)-TIM2_CH2)
- net PB8: now also U3.A2 (PB8-LTDC_B6)
- net PB9: now also U3.B3 (PB9-LTDC_B7)
- net PC2_C: now also U3.N1 (PC2_C-ADC3_INP0)
- net PC4: now also C22.1, U3.R6 (PC4-OPAMP1_VOUT)
- net PC6: now also U3.E14 (PC6-LTDC_HSYNC)
- net PC7: now also U3.D15 (PC7-LTDC_G6)
- net PC9: now also JI2C2.2 (Pin_2), R16.1, U3.E13 (PC9-I2C3_SDA)
- net PD0: now also U3.C10 (PD0-LTDC_B1)
- net PD1: now also JUART1.3 (Pin_3), U3.A10 (PD1-UART4_TX)
- net PD10: now also U3.L13 (PD10-LCD_DISP)
- net PD11: now also U3.J13 (PD11-OCTOSPIM_P1_IO0); no longer JRadio1.15 (Pin_15), JRadio1.16 (Pin_16)
- net PD12: now also U3.J15 (PD12-OCTOSPIM_P1_IO1); no longer JRadio1.13 (Pin_13), JRadio1.14 (Pin_14)
- net PD13: now also U3.H15 (PD13-OCTOSPIM_P1_IO3); no longer JRadio1.11 (Pin_11), JRadio1.12 (Pin_12)
- net PD3: now also U3.A9 (PD3-LTDC_G7)
- net PD4: now also U3.C9 (PD4-OCTOSPIM_P1_IO4)
- net PD5: now also U3.B9 (PD5-OCTOSPIM_P1_IO5)
- net PD6: now also U3.D9 (PD6-LTDC_B2)
- net PD7: now also U3.B8 (PD7-OCTOSPIM_P1_IO7)
- net PDR_ON: now also R6.1, U3.D4 (PDR_ON)
- net PE0: now also U3.B4 (PE0-LTDC_R0)
- net PE1: now also U3.C4 (PE1-LTDC_R6)
- net PE11: now also U3.R12 (PE11-LTDC_G3)
- net PE12: now also U3.P12 (PE12-LTDC_B4)
- net PE13: now also U3.P13 (PE13-LTDC_DE)
- net PE15: now also U3.P14 (PE15-LTDC_R7)
- net PE2: now also U3.C3 (PE2-OCTOSPIM_P1_IO2)
- net PF0: now also U3.F4 (PF0-OCTOSPIM_P2_IO0)
- net PF1: now also U3.F3 (PF1-OCTOSPIM_P2_IO1)
- net PF10: now also U3.K3 (PF10-OCTOSPIM_P1_CLK)
- net PF12: now also U3.P11 (PF12-OCTOSPIM_P2_DQS)
- net PF14: now also U3.R10 (PF14-I2C4_SCL)
- net PF15: now also U3.N10 (PF15-I2C4_SDA)
- net PF2: now also U3.G3 (PF2-OCTOSPIM_P2_IO2)
- net PF3: now also U3.H4 (PF3-OCTOSPIM_P2_IO3)
- net PF4: now also U3.H2 (PF4-OCTOSPIM_P2_CLK)
- net PF6: now also U3.H1 (PF6-TIM23_CH1)
- net PG0: now also U3.P8 (PG0-OCTOSPIM_P2_IO4)
- net PG1: now also U3.N9 (PG1-OCTOSPIM_P2_IO5)
- net PG10: now also U3.C8 (PG10-OCTOSPIM_P2_IO6)
- net PG11: now also U3.A7 (PG11-OCTOSPIM_P2_IO7)
- net PG12: now also U3.D8 (PG12-OCTOSPIM_P2_NCS)
- net PG14: now also U3.C7 (PG14-LTDC_B0)
- net PG15: now also U3.D7 (PG15-LCD_BL_CTRL)
- net PG2: now also U3.G15 (PG2-CTP_INT)
- net PG3: now also JFRAME1.1 (Pin_1), U3.H13 (PG3-RENDER_TIME)
- net PG6: now also U3.F14 (PG6-OCTOSPIM_P1_NCS)
- net PG7: now also R24.2, U3.G13 (PG7-LTDC_CLK)
- net PG9: now also U3.A8 (PG9-OCTOSPIM_P1_IO6)
- net PH0: now also U3.J1 (PH0-OSC_IN-RCC_OSC_IN)
- net PH10: now also U3.N14 (PH10-LTDC_R4)
- net PH11: now also U3.M13 (PH11-LTDC_R5)
- net PH12: now also U3.N15 (PH12-NRXTX)
- net PH14: now also U3.B12 (PH14-UART4_RX)
- net PH15: now also U3.D12 (PH15-LTDC_G4)
- net PH3: now also U3.R4 (PH3-LTDC_R1)
- net PH4: now also U3.P4 (PH4-LTDC_G5)
- net PH6: now also U3.P15 (PH6-LCD_RST)
- net PH8: now also U3.N13 (PH8-LTDC_R2)
- net PH9: now also U3.M14 (PH9-LTDC_R3)
- net VDDSMPS: now also U3.G1 (VDDSMPS)
- net VDD_SDC: now also C18.2, C34.2, C38.2, U3.A13 (VDDLDO), U3.A14 (VCAP), U3.A3 (VDDLDO), U3.A4 (VCAP), U3.G2 (VFBSMPS), U3.R13 (VCAP), U3.R14 (VDDLDO)
- net VLXSMPS: now also U3.F1 (VLXSMPS)
- net at JP3.3 (B): now also U3.M3 (VREF+)
- net at FB2.2: now also U3.M4 (VDDA)
- net ??: no longer names the net of J1.32
- net ??: now also R24.1
- net PD15 renamed PG5
- net PG5: now also U3.F15 (PG5-RXTX)
- net PF11 renamed PA0_C
- net PA0_C: now also U3.R3 (PA0_C-ADC1_INP0)
- net PF13 renamed PA1_C
- net PA1_C: now also U3.P3 (PA1_C-ADC2_INP1)
- net PF7 renamed PG13
- net PG13: now also U3.B7 (PG13-TIM23_CH2)
- new net: TP_OSC_.1, U3.K1 (PH1-OSC_OUT-RCC_OSC_OUT)
- new net PA12: JRadio1.11 (Pin_11), JRadio1.12 (Pin_12), U3.B15 (PA12-LSBUSB)
- new net PB14: JFRAME1.3 (Pin_3), U3.K15 (PB14-FRAME_RATE)
- new net PC13: JGPIO1.3 (Pin_3), U3.C1 (PC13-GPIO_PC13)
- new net PE4: JGPIO1.2 (Pin_2), U3.B1 (PE4-GPIO_PE4)
- new net PH7: JI2C2.3 (Pin_3), R19.1, U3.M11 (PH7-I2C3_SCL)
- no-connect marks 38 -> 66
Other:
- note added: "DAC1: 2: OUT1 via OPAMP1 PC4 3: OUT2 PA5"
- note added: "I2C3: 2: SDA PC9 3: SCL PH7"
- note added: "LCD TFT pinout equal to the DK board: CTP_INT: PG2 (39) LCD_BL_CTRL: PG15 (43) LCD_RST: PH6 (36) LCD_DISP: PD10 (24)"
- note added: "Radio Connectors: RXTX: PG5 NRXTX: PH12 LSBUSB: PA12 S0: PB12 S1: PB13 TIM23_CH1: PF6 TIM23_CH2: PG13 ADC1_INP0: PA0_C ADC2_INP1: PA1_C"
- note added: "Spare GPIO: GPIO_PE4: PE4 GPIO_PC13: PC13"
- note added: "Spare TIMER2: TIM2_CH1: PA15 TIM2_CH2: PB3"
- note added: "TGFX Frame GPIO: RENDER_TIME: PG3 MCU_ACTIVE: PB15 FRAME_RATE: PB14 VSYNC_FREQ: PA0"
- note added: "UART4: 2: RX PH14 3: TX PD1"
- note removed: "DAC1: 2: OUT1 PA4 3: OUT2 PA5"
- note removed: "I2C1: 2: SDA PB7 3: SCL PB6"
- note removed: "LCD TFT pinout equal to the DK board: CTP_INT: PG2 (39) LCD_BL_CTRL: PG15 (43) LCD_RST: instead of PH6 new PD0(36) LCD_DISP: PD10 (24)"
- note removed: "Radio Connectors: RXTX: PD15 NRXTX: PD14 LSBUSB: PD13 S0: PD12 S1: PD11 TIM23_CH1: PF6 TIM23_CH2: PF7 ADC1_INP2: PF11 ADC2_INP2: PF13"
- note removed: "UART4: 2: RX PC11 3: TX PA0"
- title: CustomSTM32H735Board -> CustomSTM32H735Board 
- moved on the sheet: C1, C10, C11, C12, C13, C14, C15, C16, C17, C19, C2, C20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
