File: CustomSTM32H735Board/KiCADFiles/CustomSTM32H735_V2_Board/CustomSTM32H735_V2_Board/_autosave-CustomSTM32H735_V2_Board.kicad_sch (KiCad schematic)
At the start: 101 parts, among them IC1 NCP700BSN33T1G, J1 FLE-125-01-G-DV, SW1 SW_Omron_B3FS, U1 L7805, U2 OPA1678IDGKT, X1 NSC5004A-25M

Commit message: local changes?
Parts:
- removed C30, C31, C35: 4.7uF low ESR, Capacitor_SMD:C_0805_2012Metric_Pad1.18x1.45mm_HandSolder, symbol Device:C
- removed FB2: FCM1608, Inductor_SMD:L_0603_1608Metric_Pad1.05x0.95mm_HandSolder, symbol Device:FerriteBead
- removed JP3: SolderJumper_3_Open, Jumper:SolderJumper-3_P1.3mm_Open_Pad1.0x1.5mm_NumberLabels, symbol Jumper:SolderJumper_3_Open
- removed R23: 1k, Resistor_SMD:R_0805_2012Metric_Pad1.20x1.40mm_HandSolder, symbol Device:R
- added C? (x3): 4.7uF low ESR, Capacitor_SMD:C_0805_2012Metric_Pad1.18x1.45mm_HandSolder, symbol Device:C
- added FB?: FCM1608, Inductor_SMD:L_0603_1608Metric_Pad1.05x0.95mm_HandSolder, symbol Device:FerriteBead
- added JP?: SolderJumper_3_Open, Jumper:SolderJumper-3_P1.3mm_Open_Pad1.0x1.5mm_NumberLabels, symbol Jumper:SolderJumper_3_Open
- added JTIM2: Conn_01x03_Socket, Connector_JST:JST_XH_B3B-XH-A_1x03_P2.50mm_Vertical, symbol Connector:Conn_01x03_Socket
- added R?: 1k, Resistor_SMD:R_0805_2012Metric_Pad1.20x1.40mm_HandSolder, symbol Device:R
Connections:
- net PB7 is gone; now on net PB11: JI2C3.2 (Pin_2), R15.1
- net PC11 is gone; now on net PH14: JUART1.2 (Pin_2)
- net +3.3V: now also JP?.1 (A), R?.2
- net GND: now also U?.F2 (VSSSMPS), U?.L4 (VREF-), U?.N3 (VSSA), C?.1, C?.1, C?.1, JTIM2.1 (Pin_1)
- net PA0: no longer JUART1.3 (Pin_3)
- net PA15: now also JTIM2.2 (Pin_2)
- net PA4: no longer C21.1
- net PB10: now also JI2C3.3 (Pin_3), R18.1; no longer JI2C2.3 (Pin_3), R17.1
- net PB11: no longer JI2C2.2 (Pin_2), R14.1
- net PB12: no longer JGPIO1.2 (Pin_2)
- net PB13: no longer JGPIO1.3 (Pin_3)
- net PB3: now also JTIM2.3 (Pin_3)
- net PB6: no longer JI2C3.3 (Pin_3), R18.1
- net PC4: now also C21.1
- net PC9: now also JI2C2.2 (Pin_2), R14.1
- net PD1: now also JUART1.3 (Pin_3)
- net PDR_ON: now also U?.D4 (PDR_ON), R?.1
- net PF12: no longer U?.P11 (PF12-TIM24_CH2)
- net VDD_SDC: now also U?.A13 (VDDLDO), U?.A14 (VCAP), U?.A3 (VDDLDO), U?.A4 (VCAP), U?.G2 (VFBSMPS), U?.R13 (VCAP), U?.R14 (VDDLDO), C?.2, C?.2, C?.2
- net at U?.M3 (VREF+): now also JP?.3 (B)
- net at U?.M4 (VDDA): now also FB?.2
- net PE4: now reaches U?.B1 (PE4)
- net PE4: now also JGPIO1.2 (Pin_2)
- net PC13: now reaches U?.C1 (PC13)
- net PC13: now also JGPIO1.3 (Pin_3)
- net PF11: no longer names the net of U?.N7 (PF11-TIM24_CH1)
- net PF11: no longer JRadio1.19 (Pin_19)
- net PF13 renamed PA1_C
- net PF7 renamed PG13
- new net: FB?.1, JP?.2 (C)
- new net PA0_C: JRadio1.19 (Pin_19)
- new net PH7: JI2C2.3 (Pin_3), R17.1
- no-connect marks 38 -> 18
Other:
- note added: "DAC1: 2: OUT1 via OPAMP PC4 3: OUT2 PA5"
- note added: "I2C3: 2: SDA PC9 3: SCL PH7"
- note added: "Radio Connectors: RXTX: PD15 NRXTX: PD14 LSBUSB: PD13 S0: PD12 S1: PD11 TIM23_CH1: PF6 TIM23_CH2: PG13 ADC1_INP0: PA0_C ADC2_INP1: PA1_C"
- note added: "Spare GPIO: GPIO_PE4: PE4 GPIO_PC13: PC13"
- note added: "Spare TIMER2: TIM2_CH1: PA15 TIM2_CH2: PB3"
- note added: "UART4: 2: RX PH14 3: TX PD1"
- note removed: "DAC1: 2: OUT1 PA4 3: OUT2 PA5"
- note removed: "I2C1: 2: SDA PB7 3: SCL PB6"
- note removed: "Radio Connectors: RXTX: PD15 NRXTX: PD14 LSBUSB: PD13 S0: PD12 S1: PD11 TIM23_CH1: PF6 TIM23_CH2: PF7 ADC1_INP2: PF11 ADC2_INP2: PF13"
- note removed: "UART4: 2: RX PC11 3: TX PA0"
- moved on the sheet: C23, C24, C27, FB1, L2, TP4, TP?, U?B, U?C
