File: CustomSTM32H735Board/KiCADFiles/CustomSTM32H735_V2_Board/CustomSTM32H735_V2_Board/CustomSTM32H735_V2_Board.kicad_pcb (KiCad board)
At the start: 4 copper layers, 127 x 73 mm, 99 parts, among them IC1 NCP700BSN33T1G, U1 L7805, U2 OPA1678IDGKT, U3 STM32H735IGT6, X1 NSC5004A-25M

Commit message: board schematics V2 checked and final
Parts:
- removed the C30 at (128.8, 109.2)
- removed the C31 at (133.3, 77.2)
- removed the C35 at (113.5, 77.7)
- removed the R22 at (141.0, 98.8)
- removed the R23 at (106.9, 78.7)
- added C17: 4.7uF low ESR, Capacitor_SMD:C_0805_2012Metric_Pad1.18x1.45mm_HandSolder, F.Cu at (36.1, 62.0)
- added C34: 4.7uF low ESR, Capacitor_SMD:C_0805_2012Metric_Pad1.18x1.45mm_HandSolder, F.Cu at (36.1, 65.0)
- added C38: 4.7uF low ESR, Capacitor_SMD:C_0805_2012Metric_Pad1.18x1.45mm_HandSolder, F.Cu at (36.1, 68.1)
- added JTIM1: Conn_01x03_Socket, Connector_JST:JST_XH_B3B-XH-A_1x03_P2.50mm_Vertical, F.Cu at (25.3, 52.6)
- added R5: 5k1, Resistor_SMD:R_0805_2012Metric_Pad1.20x1.40mm_HandSolder, F.Cu at (36.2, 50.7)
- added R6: 10k, Resistor_SMD:R_0805_2012Metric_Pad1.20x1.40mm_HandSolder, F.Cu at (36.2, 53.6)
- C1: renamed from C8; moved to B.Cu
- C12: renamed from C18; moved to B.Cu
- C2: renamed from C9; moved to B.Cu
- C28: renamed from C27; moved to B.Cu
- C29: renamed from C24; moved to B.Cu
- C30: renamed from C23; moved to B.Cu
- FB1, L2, R4, TP4, X1: moved to B.Cu
- JSWD1: renamed from JSWD; moved to B.Cu
- SW1: renamed from SW; moved to B.Cu
- U1: footprint Package_TO_SOT_THT:TO-220-3_Horizontal_TabDown -> Private:TO-220-3_Horizontal_TabDown_GND_Pad
- U3: value STM32H735IGT6 -> STM32H735IGK6; footprint Private:LQFP176_STM32H735IGT6_STM-M -> Private:BGA_735IGK6_STM; moved to B.Cu
- moved JP3 76.9 mm to (36.5, 58.8)
- moved FB2 76.3 mm to (40.6, 61.8)
- moved TP5 51.6 mm to (40.4, 64.8)
- moved X1 10.7 mm to (94.6, 96.2), turned to 180 degrees
- moved U3 10.0 mm to (113.3, 91.9), turned to 180 degrees
- moved L2 9.92 mm to (95.0, 90.9), turned to 180 degrees
- moved R4 9.79 mm to (95.1, 93.2), turned to 0 degrees
- moved C30 9.72 mm to (95.1, 84.9), turned to 0 degrees
- moved FB1 9.72 mm to (95.1, 86.9), turned to 180 degrees
- moved C28 9.70 mm to (95.1, 88.7), turned to 180 degrees
- moved C14 6.60 mm to (135.4, 91.9)
- moved R1 6.60 mm to (128.3, 84.8)
- moved UHYPERRAM1 6.60 mm to (130.0, 92.7)
- moved C11 6.60 mm to (134.1, 99.0)
- moved C8 6.60 mm to (128.0, 99.0)
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- renumbered C14 to C10, C16 to C11, C5 to C13, C20 to C14, C6 to C15, C7 to C16, C13 to C18, C15 to C19, C17 to C20, C19 to C21, C21 to C22, C22 to C23, C25 to C24, C26 to C25, C28 to C26, C29 to C27, C1 to C3, C32 to C31, C33 to C32, C34 to C33, C36 to C35, C37 to C36, C38 to C37, C2 to C4, C3 to C5, C10 to C6, C4 to C7, C11 to C8, C12 to C9, JLCD to J1, JADC to JADC1, JDAC to JDAC1, JI2C to JI2C1, JI2C to JI2C2, JI2C to JI2C3, JPOWER to JPOWER1, JUART to JUART1, R8 to R10, R9 to R11, R10 to R12, R11 to R13, R12 to R14, R13 to R15, R14 to R16, R15 to R17, R16 to R18, R17 to R19, R18 to R20, R19 to R21, R20 to R22, R21 to R23, R5 to R7, R6 to R8, R7 to R9
Connections:
- C22 pad 1: /PA4 -> /PC4
- FB2 pad 2: Net-(FB2-Pad2) -> Net-(U3B-VDDA)
- J1 pad 11: /PA11 -> /PH10
- J1 pad 12: /PJ11 -> /PH15
- J1 pad 13: /PA9 -> /PH11
- J1 pad 14: /PC1 -> /PH4
- J1 pad 15: /PB1 -> /PE1
- J1 pad 16: /PK1 -> /PC7
- J1 pad 17: /PC4 -> /PE15
- J1 pad 18: /PB15 -> /PD3
- J1 pad 21: /PE4 -> /PG14
- J1 pad 22: /PF10 -> /PE13
- J1 pad 23: /PA10 -> /PD0
- J1 pad 25: /PC9 -> /PD6
- J1 pad 28: /PA7 -> /PA4
- J1 pad 3: /PG13 -> /PE0
- J1 pad 32: /PE14 -> /??
- J1 pad 33: /PA15 -> /PB8
- J1 pad 35: /PD2 -> /PB9
- J1 pad 4: /PE5 -> /PB1
- J1 pad 5: /PA2 -> /PH3
- J1 pad 6: /PE6 -> /PB0
- J1 pad 7: /PA1 -> /PH8
- J1 pad 8: /PC0 -> /PA6
- J1 pad 9: /PB0 -> /PH9
- JGPIO1 pad 2: /PB12 -> /PE4
- JGPIO1 pad 3: /PB13 -> /PC13
- JI2C2 pad 2: /PB11 -> /PC9
- JI2C2 pad 3: /PB10 -> /PH7
- JI2C3 pad 2: /PB7 -> /PB11
- JI2C3 pad 3: /PB6 -> /PB10
- JP4 pad 3: /PD0 -> /P??
- JRadio1 pad 18: /PF7 -> /PG13
- JRadio1 pad 19: /PF11 -> /PA0_C
- JRadio1 pad 20: /PF13 -> /PA1_C
- JUART1 pad 2: /PC11 -> /PH14
- JUART1 pad 3: /PA0 -> /PD1
- R16 pad 1: /PB11 -> /PC9
- R17 pad 1: /PB7 -> /PB11
- R19 pad 1: /PB10 -> /PH7
- R20 pad 1: /PB6 -> /PB10
- UFLASH1 pad B2: /PB2 -> /PF10
- UFLASH1 pad C3: /PC5 -> /PB2
- UFLASH1 pad D2: /PF9 -> /PD12
- UFLASH1 pad D3: /PF8 -> /PD11
- UFLASH1 pad D4: /PA6 -> /PD13
- UFLASH1 pad D5: /PE7 -> /PD4
- UFLASH1 pad E1: /PE10 -> /PED7
- UFLASH1 pad E2: /PC3_C -> /PG9
- UFLASH1 pad E3: /PE8 -> /PD5
Routing:
- net +5V: track 178.1 -> 0.00 mm, vias 3 -> 0
- net GND: track 174.7 -> 0.00 mm, vias 78 -> 0
- net /PF15: track 143.0 -> 0.00 mm, vias 1 -> 0
- net /NRST: track 126.6 -> 0.00 mm, vias 2 -> 0
- net /PF14: track 101.4 -> 0.00 mm, vias 2 -> 0
- net /VDD_SDC: track 98.3 -> 0.00 mm, vias 3 -> 0
- net /PA0: track 89.3 -> 0.00 mm, vias 1 -> 0
- net /PB10: track 80.7 -> 0.00 mm, vias 1 -> 0
- net /PC2_C: track 79.2 -> 0.00 mm
- net /PF6: track 78.8 -> 0.00 mm, vias 1 -> 0
- net /PF7: track 78.6 -> 0.00 mm, vias 1 -> 0
- net /PB11: track 75.6 -> 0.00 mm, vias 1 -> 0
- net /PF13: track 75.0 -> 0.00 mm, vias 1 -> 0
- net +3.3V: track 74.9 -> 0.00 mm, vias 56 -> 0
- net /PF11: track 73.8 -> 0.00 mm, vias 1 -> 0
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- removed copper zone on In2.Cu, net +3.3V
- removed copper zone on B.Cu, net GND
- removed copper zone on F.Cu, net GND
- removed copper zone on In1.Cu, net GND
Other:
- board text added: "Stefan Meyre, HB9GZE, CPU rev. 2.0"
- board text removed: "Stefan Meyre, HB9GZE, CPU rev. 1.0"

Commit message: Final 6 Layer Board
Parts:
- added H5: MountingHole_Pad, MountingHole:MountingHole_3.2mm_M3_Pad_TopBottom, F.Cu at (105.3, 98.4)
- added JFRAME1: Conn_01x04_Socket, Connector_JST:JST_XH_B4B-XH-A_1x04_P2.50mm_Vertical, B.Cu at (196.9, 97.6)
- added R24: 0R, Resistor_SMD:R_0805_2012Metric_Pad1.20x1.40mm_HandSolder, F.Cu at (141.9, 52.1)
- C15, C16, C21, C3, C4: footprint Capacitor_Tantalum_SMD:CP_EIA-7343-30_AVX-N_Pad2.25x2.55mm_HandSolder -> Capacitor_Tantalum_SMD:CP_EIA-6032-20_AVX-F_Pad2.25x2.35mm_HandSolder
- C17: renamed from C18; footprint Capacitor_Tantalum_SMD:CP_EIA-7343-30_AVX-N_Pad2.25x2.55mm_HandSolder -> Capacitor_Tantalum_SMD:CP_EIA-6032-20_AVX-F_Pad2.25x2.35mm_HandSolder
- C18: renamed from C17; moved to B.Cu
- C31, C32, C33, C34, C38, FB2, JP3, JTIM1, R21, R22, R23, R5, R6: moved to B.Cu
- TP_VDD_SDC_1: renamed from TP4; moved to F.Cu
- moved JTIM1 181.0 mm to (196.9, 110.2), turned to 90 degrees
- moved C34 122.5 mm to (156.0, 90.0), turned to 180 degrees
- moved C38 120.1 mm to (156.0, 74.1), turned to 180 degrees
- moved R5 112.2 mm to (139.4, 94.5), turned to -90 degrees
- moved R6 108.6 mm to (136.8, 94.6), turned to -90 degrees
- moved C18 105.5 mm to (137.8, 90.0)
- moved JP3 97.4 mm to (132.9, 72.1)
- moved FB2 93.8 mm to (133.6, 74.4)
- moved R3 57.7 mm to (154.3, 103.3), turned to 180 degrees
- moved R10 56.2 mm to (190.1, 80.8)
- moved R12 56.2 mm to (192.4, 80.8)
- moved R14 55.8 mm to (191.6, 76.0)
- moved C25 55.8 mm to (193.9, 76.0)
- moved C22 55.8 mm to (172.0, 73.7)
- moved C23 55.8 mm to (186.0, 72.7)
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- renumbered C7 to C6, C6 to C7, JI2C3 to I2C2_1, JI2C2 to I2C3_1, JI2C1 to I2C4_1, TP5 to TP4
Connections:
- J1 pad 32: /?? -> Net-(J1-Pad32)
- JP4 pad 3: /P?? -> /PH6
- JRadio1 pad 10: /PD14 -> /PH12
- JRadio1 pad 11: /PD13 -> /PA12
- JRadio1 pad 12: /PD13 -> /PA12
- JRadio1 pad 13: /PD12 -> /PB12
- JRadio1 pad 14: /PD12 -> /PB13
- JRadio1 pad 15: /PD11 -> /PB12
- JRadio1 pad 16: /PD11 -> /PB13
- JRadio1 pad 3: /PD15 -> /PG5
- JRadio1 pad 4: /PD15 -> /PG5
- JRadio1 pad 5: /PD15 -> /PG5
- JRadio1 pad 6: /PD15 -> /PG5
- JRadio1 pad 7: /PD14 -> /PH12
- JRadio1 pad 8: /PD14 -> /PH12
- JRadio1 pad 9: /PD14 -> /PH12
- U1 pad 4: (no net) -> GND
- U3 pad A5: /PB6 -> unconnected-(U3A-PB6-PadA5)
- U3 pad B7: unconnected-(U3A-PG13-TIM23_CH2-PadB7) -> /PG13
- U3 pad C12: /PC10 -> unconnected-(U3C-PC10-PadC12)
- U3 pad K1: /PH1 -> unconnected-(U3B-PH1-OSC_OUT-RCC_OSC_OUT-PadK1)
- U3 pad M10: unconnected-(U3C-VSS-PadM10) -> GND
- U3 pad M7: /PC5 -> unconnected-(U3B-PC5-PadM7)
- U3 pad N12: /PH10 -> /PB10
- UFLASH1 pad E1: /PED7 -> /PD7
Routing:
- net GND: track 0.00 -> 455.6 mm, vias 0 -> 60
- net /NRST: track 0.00 -> 249.2 mm, vias 0 -> 4
- net +5V: track 0.00 -> 217.6 mm, vias 0 -> 3
- net +3.3V: track 0.00 -> 154.1 mm, vias 0 -> 24
- net /PF6: track 0.00 -> 111.2 mm, vias 0 -> 1
- net /PA1_C: track 0.00 -> 110.5 mm, vias 0 -> 2
- net /PC2_C: track 0.00 -> 107.7 mm, vias 0 -> 4
- net /PH14: track 0.00 -> 106.1 mm, vias 0 -> 2
- net /PB15: track 0.00 -> 103.8 mm, vias 0 -> 2
- net /VDD_SDC: track 0.00 -> 103.2 mm, vias 0 -> 6
- net /PC13: track 0.00 -> 101.9 mm, vias 0 -> 1
- net /PA0_C: track 0.00 -> 100.7 mm, vias 0 -> 2
- net /PF15: track 0.00 -> 88.4 mm, vias 0 -> 5
- net /PF14: track 0.00 -> 87.0 mm, vias 0 -> 4
- net /PA0: track 0.00 -> 83.8 mm, vias 0 -> 1
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- added copper zone on In2.Cu, net +3.3V
- added copper zone on In1.Cu, net GND
