File: CustomSTM32H735Board/KiCADFiles/CustomSTM32H735_V2_1_Board/CustomSTM32H735_V2_1_Board/CustomSTM32H735_V2_1_Board.kicad_pcb (KiCad board)
At the start: 6 copper layers, 127 x 73 mm, 108 parts, among them IC1 NCP700BSN33T1G, J1 FLE-125-01-G-DV, SW1 SW_Omron_B3FS, U1 L7805, U2 OPA1678IDGKT, U3 STM32H735IGK6, X1 NSC5004A-25M

Commit message: finished v2.1 and send off to JLCPCB
Parts:
- moved C37 33.1 mm to (130.6, 52.9), turned to 180 degrees
- renumbered TP_VDD_SDC to TP_VDD_SDC_1
Routing:
- net GND: track 375.1 -> 378.1 mm, vias 62 -> 64
- net +3.3V: track 84.6 -> 85.4 mm, vias 38 -> 37
Other:
- board text added: "+"
- board text added: "-"
- board text added: "1 2"
- board text added: "1,2 GND 3,4,5,6 RXTX PG5 7,8,9,10 NRXTX PH12 11,12 LSBUSB PA12 13,15 S0 PB12 14,16 S1 PB13 17 TIM23_CH1 PF6 18 TIM23_CH2 PG13 19 ADC1_INP0 PA0_C 20 ADC2_INP1 PA1_C"
- board text added: "19 20"
