File: KiCAD Files/Mixer2/Mixer2/Mixer2.kicad_sch (KiCad schematic)
At the start: 83 parts, among them IC1 FST3253MTCX, K1 G6K-2F-Y DC3, U1 BGA420H6327XTSA1, U2 Si5351A-B-GT, U3 SN74AC74PWR, U4 TXU0101DBVR, U5 4053, U6 4053, U7 OPA1678IDGKT, U8 OPA1678IDGKT, U9 OPA1678IDGKT, Y1 ECS-250-8-30B-CKM

Commit message: final mixer2 board
Parts:
- removed Tx1, TxN1: TestPoint, Connector_Pin:Pin_D0.7mm_L6.5mm_W1.8mm_FlatFork, symbol Connector:TestPoint
- added C10, C21: 100nF, Capacitor_SMD:C_0603_1608Metric_Pad1.08x0.95mm_HandSolder, symbol Device:C
- R16: renamed from R22; value 1k -> 10k
- R17: renamed from R23; value 1k -> 10k
- R5: renamed from R4; value 47R -> DNF
- renumbered C3 to C1, C10 to C11, C11 to C12, C12 to C13, C13 to C14, C14 to C15, C15 to C16, C16 to C17, C19 to C18, C17 to C19, C1 to C2, C18 to C20, C20 to C23, C21 to C24, C2 to C3, C9 to C6, C6 to C7, C7 to C8, C8 to C9, R16 to R18, R17 to R19, R18 to R20, R19 to R21, R20 to R22, R21 to R23, R5 to R4, R8 to R6, R6 to R7, R7 to R8, Tx2 to Tx1, U3 to U2, U2 to U3
Connections:
- net +3.3V: now also C21.2
- net GND: now also C21.1
- net SI5351CLK: now also C10.2; no longer U4.4 (BY)
- new net: C10.1, U4.4 (BY)
Other:
- moved on the sheet: C1, C11, C12, C13, C14, C19, C2, C20, C22, C23, C24, C3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

Commit message: Very fianl Version 1.0 working well
Parts:
- C3: value 100nF -> 1.5nF
Changed lines of the file:
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@@
 			)
 		)
-		(property "Value" "100nF"
+		(property "Value" "1.5nF"
 			(at 85.09 227.33 90)
 			(effects
