File: KiCAD Files/Mixer/Mixer/Mixer.kicad_pcb (KiCad board)
At the start: 4 copper layers, 59 x 30.5 mm, 71 parts, among them IC1 FST3253MTCX, J1 Conn_01x02_Socket, J2 Conn_01x04_Socket, K1 G6K-2F-Y DC3, U1 OPA1678IDGKT, U2 SN74AC74PWR, U3 OPA1678IDGKT, U4 OPA1678IDGKT, U5 NC7SZ04P5X, U6 4053, U7 4053

Commit message: minor
Parts:
- added C1: 100nF, Capacitor_SMD:C_0603_1608Metric_Pad1.08x0.95mm_HandSolder, B.Cu at (108.2, 57.9)
- added C4: 100nF, Capacitor_SMD:C_0603_1608Metric_Pad1.08x0.95mm_HandSolder, B.Cu at (105.3, 56.9)
- added C8: 1uF, Capacitor_SMD:C_0805_2012Metric_Pad1.18x1.45mm_HandSolder, B.Cu at (108.5, 52.0)
- added C9: 100nF, Capacitor_SMD:C_0603_1608Metric_Pad1.08x0.95mm_HandSolder, B.Cu at (111.5, 52.6)
- added L3: 100u, Inductor_SMD:L_0805_2012Metric_Pad1.15x1.40mm_HandSolder, B.Cu at (114.4, 52.6)
- added U1: BGA420H6327XTSA1, Private:PG-SOT343-4-1_INF, B.Cu at (108.6, 54.9)
- C12: renamed from C6; footprint Capacitor_SMD:C_0805_2012Metric_Pad1.18x1.45mm_HandSolder -> Capacitor_SMD:C_0603_1608Metric_Pad1.08x0.95mm_HandSolder
- R5: renamed from R1; footprint Resistor_SMD:R_0805_2012Metric_Pad1.20x1.40mm_HandSolder -> Resistor_SMD:R_0603_1608Metric_Pad0.98x0.95mm_HandSolder
- R8: renamed from R6; footprint Resistor_SMD:R_0805_2012Metric_Pad1.20x1.40mm_HandSolder -> Resistor_SMD:R_0603_1608Metric_Pad0.98x0.95mm_HandSolder
- moved R8 0.33 mm to (115.5, 70.2)
- moved R5 0.33 mm to (115.4, 74.1)
- moved C12 0.06 mm to (115.4, 78.3)
- renumbered C8 to C10, C13 to C11, C9 to C13, C10 to C14, C11 to C15, C12 to C16, C7 to C17, C14 to C18, C15 to C19, C16 to C20, C17 to C21, C18 to C22, C19 to C23, C20 to C24, C21 to C25, C1 to C3, C3 to C5, C4 to C6, C5 to C7, J1 to Clock_In, I_In_Tx1 to I_In_Tx, I_Out_Rx1 to I_Out_Rx, J2 to J1, Q_In_Tx1 to Q_In_Tx, Q_Out_Rx1 to Q_Out_Rx, R2 to R1, R3 to R2, R4 to R3, R5 to R4, R7 to R6, R8 to R7, RF_In1 to RF_In, RF_Out1 to RF_Out, Supply1 to Supply, Tx1 to Tx, TxN1 to TxN, U1 to U2, U2 to U5, U5 to U8
Connections:
- IC1 pad 14: /Clk_S0 -> /S0
- K1 pad 4: /RF_Out -> Net-(C1-Pad1)
Routing:
- net /Clk_S0: track 36.0 -> 14.8 mm, vias 1 -> 0
- net /S0: track 2.93 -> 22.5 mm, vias 0 -> 2
- net Net-(U1-VD): track 0.00 -> 6.28 mm
- net Net-(C1-Pad1): track 0.00 -> 4.42 mm
- net Net-(U1-OUT): track 0.00 -> 3.54 mm
- net Net-(U1-IN): track 0.00 -> 2.00 mm
- net /Tx: track 34.4 -> 35.9 mm
- net +5V: track 36.9 -> 38.3 mm, vias 13 -> 14
- added copper zone on In2.Cu, net +5V
- removed copper zone on In1.Cu, net GND
