File: KiCAD Files/Mixer/Mixer/Mixer.kicad_sch (KiCad schematic)
At the start: 71 parts, among them IC1 FST3253MTCX, J1 Conn_01x02_Socket, J2 Conn_01x04_Socket, K1 G6K-2F-Y DC3, U1 OPA1678IDGKT, U2 SN74AC74PWR, U3 OPA1678IDGKT, U4 OPA1678IDGKT, U5 NC7SZ04P5X, U6 4053, U7 4053

Commit message: minor
Parts:
- added C1, C4, C9: 100nF, Capacitor_SMD:C_0603_1608Metric_Pad1.08x0.95mm_HandSolder, symbol Device:C
- added C8: 1uF, Capacitor_SMD:C_0805_2012Metric_Pad1.18x1.45mm_HandSolder, symbol Device:C
- added L3: 100u, Inductor_SMD:L_0805_2012Metric_Pad1.15x1.40mm_HandSolder, symbol Device:L
- added U1: BGA420H6327XTSA1, Private:PG-SOT343-4-1_INF, symbol Private:BGA420H6327XTSA1
- C12: renamed from C6; footprint Capacitor_SMD:C_0805_2012Metric_Pad1.18x1.45mm_HandSolder -> Capacitor_SMD:C_0603_1608Metric_Pad1.08x0.95mm_HandSolder
- R5: renamed from R1; footprint Resistor_SMD:R_0805_2012Metric_Pad1.20x1.40mm_HandSolder -> Resistor_SMD:R_0603_1608Metric_Pad0.98x0.95mm_HandSolder
- R8: renamed from R6; footprint Resistor_SMD:R_0805_2012Metric_Pad1.20x1.40mm_HandSolder -> Resistor_SMD:R_0603_1608Metric_Pad0.98x0.95mm_HandSolder
- renumbered C8 to C10, C13 to C11, C9 to C13, C10 to C14, C11 to C15, C12 to C16, C7 to C17, C14 to C18, C15 to C19, C16 to C20, C17 to C21, C18 to C22, C19 to C23, C20 to C24, C21 to C25, C1 to C3, C3 to C5, C4 to C6, C5 to C7, J1 to Clock_In1, J2 to J1, R2 to R1, R3 to R2, R4 to R3, R5 to R4, R7 to R6, R8 to R7, U1 to U2, U2 to U5, U5 to U8
Connections:
- net +5V: now also L3.1
- net GND: now also C8.1, C9.1, U1.2 (GND)
- net RF_Out: now also C4.2; no longer K1.4
- new net: C1.1, K1.4
- new net: C1.2, U1.1 (IN)
- new net: C8.2, C9.2, L3.2, U1.4 (VD)
- new net: C4.1, U1.3 (OUT)
Other:
- note added: "instead of 4x 1uF use 47R"
- moved on the sheet: C11, C12, C13, C14, C15, C16, C17, C18, C19, C20, C21, C3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
